File: PCB/Riddler-Datapack/power.kicad_sch (KiCad schematic)
At the start: 26 parts, among them J1 UJ20-C-H-G-SMT-1-P16-TR, P1 S2B-PH-SM4-TB, Q1 BC847W, Q2 AO3401A, U2 USBLC6-2P6, U3 TLV62568DBV, U5 BQ25170DSGR

Commit message: Complete schematics v0.5, add schematic PDF export and active prop reference
Parts:
- added C4: 4.7u, Capacitor_SMD:C_0603_1608Metric, symbol Device:C
- added C7: 10u, Capacitor_SMD:C_0603_1608Metric, symbol Device:C
- added L2: 1u, Inductor_SMD:L_1008_2520Metric, symbol Device:L
- added R10: 73.2k, Resistor_SMD:R_0402_1005Metric, symbol Device:R
- added R11: 10k, Resistor_SMD:R_0402_1005Metric, symbol Device:R
- added U4: TPS61023DRLR, TPS61023DRLR:SOT563-ORI, symbol TPS61023DRLR:TPS61023DRLR
- renumbered C9 to C1, C10 to C2, C11 to C3, C2 to C5, D2 to D1, D1 to D2, Q2 to Q1, Q1 to Q2, R9 to R1, R5 to R2, R6 to R3, R2 to R4, R1 to R5, R8 to R6, R3 to R8, R4 to R9, U2 to U1, U5 to U2
Connections:
- net GND: now also C4.2, C7.2, R11.1, U4.4 (GND)
- net VBAT: now also C4.1, L2.1, U4.3 (VIN)
- net BAT_STAT: no longer names the net of D1.1 (K), U2.5 (STAT)
- new net: R10.1, R11.2, U4.1 (FB)
- new net: L2.2, U4.5 (SW)
- new net +5V: C7.1, R10.2, U4.6 (VOUT)
- new net EN_5V: U4.2 (EN)
Other:
- note added: "ATTENTION FOR L1 & L2: I HIGHLY RECOMMAND USING A SHIELDED COIL TO REDUCE EMI"
- note added: "DCDC: 5V / 1A"
- note removed: "ATTENTION FOR L1: I HIGHLY RECOMMAND USING A SHIELDED COIL TO REDUCE EMI"
- moved on the sheet: C5, C6, L1, Q1, Q2, R6, R7, R8, R9, U3
