File: PCB/Mini Version/Riddler-Datapack mini/power.kicad_sch (KiCad schematic)
At the start: 11 parts, among them J1 UJ20-C-H-G-SMT-1-P16-TR, U1 USBLC6-2P6, U3 TLV62568DBV

Commit message: feat(hardware): complete 4-layer PCB routing for Mini Datapack prop and add 3D exports
Other:
- note added: "ATTENTION FOR L1: I HIGHLY RECOMMAND USING A SHIELDED COIL TO REDUCE EMI"
- note removed: "ATTENTION FOR L1 & L2: I HIGHLY RECOMMAND USING A SHIELDED COIL TO REDUCE EMI"
Changed lines of the file:
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@@
 		)
 	)
-	(text "ATTENTION FOR L1 & L2: \nI HIGHLY RECOMMAND \nUSING A SHIELDED COIL\nTO REDUCE EMI"
+	(text "ATTENTION FOR L1: \nI HIGHLY RECOMMAND \nUSING A SHIELDED COIL\nTO REDUCE EMI"
 		(exclude_from_sim no)
 		(at 115.57 38.1 0)
