File: PCB/Mini Version/Riddler-Datapack mini/peripherals.kicad_sch (KiCad schematic)
At the start: 29 parts, among them J2 DISPLAY, J4 Micro_SD_Card

Commit message: feat(hardware): complete 4-layer PCB routing for Mini Datapack prop and add 3D exports
Parts:
- removed D10, D11, D12, D3, D4, D5, D6, D7, D8, D9: WS2812B, LED_SMD:LED_WS2812B_PLCC4_5.0x5.0mm_P3.2mm, symbol LED:WS2812B
- added C28, C29: 100n, Capacitor_SMD:C_0402_1005Metric, symbol Device:C
- added D1, D10, D11, D12, D13, D3, D4, D5, D6, D7, D8, D9: WS2812B-2020, LED_SMD:LED_WS2812B-2020_PLCC4_2.0x2.0mm, symbol LED:WS2812B-2020
Connections:
- net +3V3: now also C28.1, C29.1, D1.4 (VDD), D10.4 (VDD), D11.4 (VDD), D12.4 (VDD), D13.4 (VDD), D3.4 (VDD), D4.4 (VDD), D5.4 (VDD), D6.4 (VDD), D7.4 (VDD), D8.4 (VDD), D9.4 (VDD)
- net GND: now also C28.2, C29.2, D1.2 (VSS), D10.2 (VSS), D11.2 (VSS), D12.2 (VSS), D13.2 (VSS), D3.2 (VSS), D4.2 (VSS), D5.2 (VSS), D6.2 (VSS), D7.2 (VSS), D8.2 (VSS), D9.2 (VSS)
- new net: D8.1 (DOUT), D9.3 (DIN)
- new net: D7.1 (DOUT), D8.3 (DIN)
- new net: D5.1 (DOUT), D6.3 (DIN)
- new net: D4.1 (DOUT), D5.3 (DIN)
- new net: D12.1 (DOUT), D13.3 (DIN)
- new net: D1.1 (DOUT), D3.3 (DIN)
- new net: D10.1 (DOUT), D11.3 (DIN)
- new net: D10.3 (DIN), D9.1 (DOUT)
- new net NPD_F: D12.3 (DIN)
- new net NPD_LS: D7.3 (DIN)
- new net NPD_PWRS: D4.3 (DIN)
- new net NPD_RS: D1.3 (DIN)
- no-connect marks 4 -> 7
Other:
- note added: "DCDC-SECTION"
- note added: "LEFT SIDE GRILL"
- note added: "RIGHT SIDE GRILL"
- note added: "TOP FAN GRILL"

Commit message: v1.1: update Mini Datapack with repositioned USB-C, relief vias, and v1p1 exports
Connections:
- net CS_SD2: now reaches J2.10 (Pin_10)
- net MISO: now reaches J2.5 (Pin_5)
- no-connect marks 7 -> 5
Changed lines of the file:
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@@
 	)
 	(no_connect
-		(at 228.6 53.34)
-	)
-	(no_connect
 		(at 170.18 194.31)
 	)
@@
 		(at 93.98 227.33)
 	)
-	(no_connect
-		(at 228.6 66.04)
-	)
 	(wire
 		(pts
@@
 	(wire
 		(pts
+			(xy 213.36 66.04) (xy 228.6 66.04)
+		)
+		(stroke
+			(width 0)
+			(type default)
+		)
+	)
+	(wire
+		(pts
 			(xy 43.18 41.91) (xy 43.18 52.07)
 		)
@@
 	(wire
 		(pts
+			(xy 213.36 53.34) (xy 228.6 53.34)
+		)
+		(stroke
+			(width 0)
+			(type default)
+		)
+	)
+	(wire
+		(pts
 			(xy 53.34 34.29) (xy 53.34 31.75)
 		)
@@
 		)
 	)
+	(hierarchical_label "MISO"
+		(shape output)
+		(at 213.36 53.34 180)
+		(effects
+			(font
+				(size 1.27 1.27)
+			)
+			(justify right)
+		)
+	)
 	(hierarchical_label "MOSI"
 		(shape input)
@@
 		(effects
 			(font
+				(size 1.27 1.27)
+			)
+			(justify right)
+		)
+	)
+	(hierarchical_label "CS_SD2"
+		(shape input)
+		(at 213.36 66.04 180)
+		(effects
+			(font
